Commit message: Initial project changes

File: lwr_description/urdf/ati_sensor.urdf.xacro (robot description, xacro)
@@ -14,6 +14,8 @@
 		      xyz="-0.00480740431783837 0.00412111608218374 -0.0111556038816137"
 		      rpy="0 0 0" />
-		    <mass
-		      value="${0.138+0.171+0.212}" />
+		    <!-- <mass
+		      value="${0.138+0.171+0.212}" /> -->
+        <mass
+		      value="0.1" />
 		    <inertia
 		      ixx="4.36061005979496E-05"

File: lwr_description/urdf/screwdriver.urdf.xacro (robot description, xacro)
@@ -7,5 +7,5 @@
           xyz="0.00019306 -0.00063333 -0.10165"
           rpy="0 0 0" />
-        <mass value="0.22973" />
+        <mass value="0.005" />
         <inertia
           ixx="0.00044365"
